File: src/SimLinkup/HardwareSupport/TeensyEWMU/KiCAD Project/EWMU.sch (KiCad schematic (older format))
At the start: 26 parts, among them J1 Conn_01x02, Q1 TIP127, Q2 TIP127, Q3 TIP127, Q4 TIP127, Q5 TIP127, U1 Teensy3.6

Commit message: Adding TeensyEWMU column driver board schematic and initial test firmware (just displays hard-coded string for now)
Parts:
- Dis1, Dis2, Dis3, Dis4, Dis5, Dis6, Dis7, Dis8: symbol hcms-2313:HCMS-2313 -> EWMU-rescue:HCMS-2313-hcms-2313
Changed lines of the file:
@@
 EESchema Schematic File Version 4
+LIBS:EWMU-cache
 EELAYER 29 0
 EELAYER END
@@
 	10450 700  10450 1050
 $Comp
-L hcms-2313:HCMS-2313 Dis1
+L EWMU-rescue:HCMS-2313-hcms-2313 Dis1
 U 1 1 5F667DCB
 P 1050 4500
@@
 	2000 5300 2000 5150
 $Comp
-L hcms-2313:HCMS-2313 Dis2
+L EWMU-rescue:HCMS-2313-hcms-2313 Dis2
 U 1 1 5F6A7B44
 P 2400 4500
@@
 	3250 5300 3250 5150
 $Comp
-L hcms-2313:HCMS-2313 Dis3
+L EWMU-rescue:HCMS-2313-hcms-2313 Dis3
 U 1 1 5F6AC71F
 P 3750 4500
@@
 	4600 5300 4600 5150
 $Comp
-L hcms-2313:HCMS-2313 Dis4
+L EWMU-rescue:HCMS-2313-hcms-2313 Dis4
 U 1 1 5F6AC73D
 P 5100 4500
@@
 	5950 5300 5950 5150
 $Comp
-L hcms-2313:HCMS-2313 Dis5
+L EWMU-rescue:HCMS-2313-hcms-2313 Dis5
 U 1 1 5F6B58F9
 P 1100 6200
@@
 	1950 7000 1950 6850
 $Comp
-L hcms-2313:HCMS-2313 Dis6
+L EWMU-rescue:HCMS-2313-hcms-2313 Dis6
 U 1 1 5F6B5917
 P 2450 6200
@@
 	3300 7000 3300 6850
 $Comp
-L hcms-2313:HCMS-2313 Dis7
+L EWMU-rescue:HCMS-2313-hcms-2313 Dis7
 U 1 1 5F6B5935
 P 3800 6200
@@
 	4650 7000 4650 6850
 $Comp
-L hcms-2313:HCMS-2313 Dis8
+L EWMU-rescue:HCMS-2313-hcms-2313 Dis8
 U 1 1 5F6B5953
 P 5150 6200
@@
 Wire Wire Line
 	2050 7300 2050 6850
-Text GLabel 850  3600 3    50   Output ~ 0
-GND
-Wire Wire Line
+Text GLabel 850  3600 3    50   Input ~ 0
+GND
+Wire Wire Line

Commit message: Adding TeensyEWMU column driver board schematic and initial test firmware (just displays hard-coded string for now)
Parts:
- Dis1, Dis2, Dis3, Dis4, Dis5, Dis6, Dis7, Dis8: symbol EWMU-rescue:HCMS-2313-hcms-2313 -> EWMU-rescue:HCMS-2313-hcms-2313-EWMU-rescue
Changed lines of the file:
@@
 	10450 700  10450 1050
 $Comp
-L EWMU-rescue:HCMS-2313-hcms-2313 Dis1
+L EWMU-rescue:HCMS-2313-hcms-2313-EWMU-rescue Dis1
 U 1 1 5F667DCB
 P 1050 4500
@@
 	2000 5300 2000 5150
 $Comp
-L EWMU-rescue:HCMS-2313-hcms-2313 Dis2
+L EWMU-rescue:HCMS-2313-hcms-2313-EWMU-rescue Dis2
 U 1 1 5F6A7B44
 P 2400 4500
@@
 	3250 5300 3250 5150
 $Comp
-L EWMU-rescue:HCMS-2313-hcms-2313 Dis3
+L EWMU-rescue:HCMS-2313-hcms-2313-EWMU-rescue Dis3
 U 1 1 5F6AC71F
 P 3750 4500
@@
 	4600 5300 4600 5150
 $Comp
-L EWMU-rescue:HCMS-2313-hcms-2313 Dis4
+L EWMU-rescue:HCMS-2313-hcms-2313-EWMU-rescue Dis4
 U 1 1 5F6AC73D
 P 5100 4500
@@
 	5950 5300 5950 5150
 $Comp
-L EWMU-rescue:HCMS-2313-hcms-2313 Dis5
+L EWMU-rescue:HCMS-2313-hcms-2313-EWMU-rescue Dis5
 U 1 1 5F6B58F9
 P 1100 6200
@@
 	1950 7000 1950 6850
 $Comp
-L EWMU-rescue:HCMS-2313-hcms-2313 Dis6
+L EWMU-rescue:HCMS-2313-hcms-2313-EWMU-rescue Dis6
 U 1 1 5F6B5917
 P 2450 6200
@@
 	3300 7000 3300 6850
 $Comp
-L EWMU-rescue:HCMS-2313-hcms-2313 Dis7
+L EWMU-rescue:HCMS-2313-hcms-2313-EWMU-rescue Dis7
 U 1 1 5F6B5935
 P 3800 6200
@@
 	4650 7000 4650 6850
 $Comp
-L EWMU-rescue:HCMS-2313-hcms-2313 Dis8
+L EWMU-rescue:HCMS-2313-hcms-2313-EWMU-rescue Dis8
 U 1 1 5F6B5953
 P 5150 6200
@@
 0.1
 Text Notes 10445 1075 3    50   ~ 0
+E
+Text Notes 10440 1380 3    50   ~ 0
 C
-Text Notes 10440 1380 3    50   ~ 0
-E
 Text Notes 10230 1250 0    50   ~ 0
 B
@@
 	10450 1850 10450 2200
 Text Notes 10445 2225 3    50   ~ 0
+E
+Text Notes 10440 2530 3    50   ~ 0
 C
-Text Notes 10440 2530 3    50   ~ 0
-E
 Text Notes 10230 2400 0    50   ~ 0
 B
@@
 	10450 3000 10450 3350
 Text Notes 10445 3375 3    50   ~ 0
+E
+Text Notes 10440 3680 3    50   ~ 0
 C
-Text Notes 10440 3680 3    50   ~ 0
-E
 Text Notes 10230 3550 0    50   ~ 0
 B
@@
 	10450 4150 10450 4500
 Text Notes 10445 4525 3    50   ~ 0
+E
+Text Notes 10440 4830 3    50   ~ 0
 C
-Text Notes 10440 4830 3    50   ~ 0
-E
 Text Notes 10230 4700 0    50   ~ 0
 B
@@
 	10450 5300 10450 5650
 Text Notes 10445 5675 3    50   ~ 0
+E
+Text Notes 10440 5980 3    50   ~ 0
 C
-Text Notes 10440 5980 3    50   ~ 0
-E
 Text Notes 10230 5850 0    50   ~ 0
 B
